Commit message: feat: update urdf and support mac sim2sim

File: resources/robots/t1/T1_locomotion.urdf (robot description, URDF)
Before this commit: robot T1, 24 links, 23 joints
Links:
- link Hip_Roll_Left: geometry visual mesh filename=meshes/Hip_Roll_Left.STL
- link Hip_Roll_Right: geometry visual mesh filename=meshes/Hip_Roll_Right.STL
- link Hip_Yaw_Left: geometry collision cylinder length=0.16 radius=0.05; visual mesh filename=meshes/Hip_Yaw_Left.STL
- link Hip_Yaw_Right: geometry collision cylinder length=0.16 radius=0.05; visual mesh filename=meshes/Hip_Yaw_Right.STL
- link Shank_Left: geometry collision cylinder length=0.15 radius=0.05; visual mesh filename=meshes/Shank_Left.STL
- link Shank_Right: geometry collision cylinder length=0.15 radius=0.05; visual mesh filename=meshes/Shank_Right.STL
Joints:
- joint Left_Ankle_Roll: limit lower=-0.44 upper=0.44 effort=6 velocity=12.4 -> lower=-0.44 upper=0.44 effort=15 velocity=12.4
- joint Left_Hip_Pitch: limit lower=-1.8 upper=1.57 effort=45 velocity=12.5 -> lower=-1.8 upper=1.57 effort=60 velocity=12.5
- joint Left_Hip_Roll: limit lower=-0.52 upper=1.57 effort=25 velocity=10.9 -> lower=-0.3 upper=1.57 effort=30 velocity=10.9
- joint Left_Knee_Pitch: limit lower=0 upper=2.34 effort=65 velocity=11.7 -> lower=0 upper=2.34 effort=90 velocity=11.7
- joint Right_Ankle_Roll: limit lower=-0.44 upper=0.44 effort=6 velocity=12.4 -> lower=-0.44 upper=0.44 effort=15 velocity=12.4
- joint Right_Hip_Pitch: limit lower=-1.8 upper=1.57 effort=45 velocity=12.5 -> lower=-1.8 upper=1.57 effort=60 velocity=12.5
- joint Right_Hip_Roll: limit lower=-1.57 upper=0.52 effort=25 velocity=10.9 -> lower=-1.57 upper=0.3 effort=30 velocity=10.9
- joint Right_Knee_Pitch: limit lower=0 upper=2.34 effort=65 velocity=11.7 -> lower=0 upper=2.34 effort=90 velocity=11.7
